File: 2020 Board/Clear Excess/Spring2020.brd (EAGLE design)
At the start: 193.5 x 118.1 mm, 16 parts, among them U1 TB67H401FTG(O,EL)

Commit message: Added routing
Parts:
- removed LED1: (no value), led:LED5MM
- removed R1: (no value), rcl:0309/10
- removed U$1: IL-711, Spring2016Optoisolator:8PINSOIC
- added ROSC, RRS: (no value), rcl:0309/10
- moved IMU 137.7 mm to (35.6, 38.1)
- moved REAR-MOTOR 116.6 mm to (43.2, 62.2)
- moved U1 82.4 mm to (36.8, 22.9)
- moved GND-JUMPER 82.2 mm to (12.7, 26.7), turned to 270 degrees
- moved RC 75.5 mm to (47.0, 38.1)
- moved U$2 62.1 mm to (14.0, 36.8), turned to 0 degrees
- moved C18 60.5 mm to (26.7, 45.7)
- moved C19 47.3 mm to (20.3, 45.7), turned to 0 degrees
- moved BIKE-PWR 42.7 mm to (25.4, 38.1)
- moved R18 37.0 mm to (44.5, 54.6)
- moved U$7 35.9 mm to (47.0, 48.3), turned to 0 degrees
- moved C16 35.8 mm to (33.0, 45.7), turned to 0 degrees
- moved C15 29.6 mm to (39.4, 45.7)
Connections:
- net FRONT-DIGI renamed REVERSE_IN
- removed net 24GND: BIKE-PWR.1
- removed net BGND: C15.2, C16.2, C19.2, GND-JUMPER.2, REAR-MOTOR.1, U$2.5, U$7.5
- removed net BIKE-IN: BIKE-PWR.2
- removed net FRONT-DIGIOUT: U$2.6
- removed net FRONT-PWM: U$2.2
- removed net FRONT-PWMOUT/SERVO1: U$2.7
- removed net GND1: U$1.4
- removed net GND2: U$1.5
- removed net LED1: R1.1
- removed net N$1: LED1.A, R1.2
- removed net REG5V: C16.1, C19.1, U$2.8, U$7.8
- removed net VCC: U1.34, U1.46, U1.47
- removed net VDD1: U$1.1
- removed net VDD2: U$1.8
- removed net VREFB: U1.41
- new net BKGND: BIKE-PWR.1, C15.2, C16.2, C19.2, GND-JUMPER.2, REAR-MOTOR.1, U$2.5, U$7.5, U1.15, U1.22
- new net BKPWR: BIKE-PWR.2, RRS.2, U1.32
- new net F+: U1.10, U1.11, U1.26, U1.27
- new net F-: U1.16, U1.17, U1.20, U1.21
- new net FVCC: ROSC.1, U1.34, U1.39, U1.46, U1.47
- new net N$5: ROSC.2, U1.43
- new net RS: RRS.1, U1.29, U1.30, U1.7, U1.8
- net 5V: now also C16.1, C19.1, U$2.8, U$7.8
- net GND: now also U1.18, U1.19, U1.37, U1.40, U1.41, U1.49, U1.5; no longer LED1.K
- net I_1: no longer U1.2
- net I_2: no longer U1.3
- net REVERSE: now also U$2.6
Routing:
- net CH2: track 296.5 -> 0.00 mm
- net CH6: track 245.8 -> 0.00 mm, vias 8 -> 0
- net REAR-TIMER-IN: track 218.0 -> 0.00 mm, vias 2 -> 0
- net FRONT-PWM: track 217.5 -> 0.00 mm, vias 2 -> 0
- net CH4: track 216.8 -> 0.00 mm
- net CH3: track 214.0 -> 0.00 mm, vias 6 -> 0
- net REAR-PWM: track 206.6 -> 0.00 mm, vias 4 -> 0
- net CH5: track 198.7 -> 0.00 mm, vias 4 -> 0
- net REG5V: track 159.8 -> 0.00 mm, vias 10 -> 0
- net BKGND: track 0.00 -> 96.9 mm
- net FRONT-DIGIOUT: track 89.2 -> 0.00 mm, vias 8 -> 0
- net REAR-TIMER: track 99.3 -> 16.7 mm, vias 2 -> 0
- net REAR-PWMR/SERVO2: track 96.9 -> 15.2 mm, vias 6 -> 0
- net IMU-CS: track 81.2 -> 0.00 mm, vias 6 -> 0
- net 24GND: track 73.7 -> 0.00 mm
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- removed copper zone on layer 16, net BGND
- removed copper zone on layer 16, net GND
- removed copper zone on layer 1, net HOLE
Other:
- board size 193.5 x 118.1 mm -> 100 x 80 mm
