File: 2020 Board/Clear Excess/Spring2020.sch (EAGLE design)
At the start: 16 parts, among them U1 TB67H401FTG(O,EL)

Commit message: Added routing
Parts:
- removed LED1: (no value), led:LED5MM
- removed R1: (no value), rcl:R-US_0309/10
- removed U$1: IL-711, Spring2016Optoisolator:IL-711
- added ROSC, RRS: (no value), rcl:R-US_0309/10
Connections:
- net FRONT-DIGI renamed REVERSE_IN
- removed net 24GND: BIKE-PWR-1.KL
- removed net BGND: C15.2, C16.2, C19.2, GND-JUMPER.2, REAR-MOTOR.1, U$2.GND2, U$7.GND2
- removed net BIKE-IN: BIKE-PWR-2.KL
- removed net FRONT-DIGIOUT: U$2.OUT2
- removed net FRONT-PWM: U$2.IN1
- removed net FRONT-PWMOUT/SERVO1: U$2.OUT1
- removed net LED1: R1.1
- removed net N$1: LED1.A, R1.2
- removed net REG5V: C16.1, C19.1, U$2.VDD2, U$7.VDD2
- removed net VCC: U1.PWMA, U1.PWMB, U1.VCC
- new net BKGND: BIKE-PWR-1.KL, C15.2, C16.2, C19.2, GND-JUMPER.2, REAR-MOTOR.1, U$2.GND2, U$7.GND2, U1.GND_3, U1.GND_6
- new net BKPWR: BIKE-PWR-2.KL, RRS.2, U1.VM
- new net F+: U1.OUTA+, U1.OUTA+_2, U1.OUTB+, U1.OUTB+_2
- new net F-: U1.OUTA-, U1.OUTA-_2, U1.OUTB-, U1.OUTB-_2
- new net FVCC: ROSC.1, U1.HBMODE, U1.PWMA, U1.PWMB, U1.VCC
- new net N$5: ROSC.2, U1.OSCM
- new net RS: RRS.1, U1.RSA, U1.RSA_2, U1.RSB, U1.RSB_2
- net 5V: now also C16.1, C19.1, U$2.VDD2, U$7.VDD2
- net GND: now also U1.FBB, U1.GND, U1.GND_2, U1.GND_4, U1.GND_5, U1.GND_7, U1.VREFB; no longer LED1.C
- net I_1: no longer U1.INB1
- net I_2: no longer U1.INB2
- net REVERSE: now also U$2.OUT2
Other:
- moved on the sheet: C16
